Commit message: Merged urdf

File: ros2_robot_ws/src/eg2_4b_description/urdf/eg2_4b_description.urdf (robot description, URDF)
Before this commit: robot eg2_4b_description, 5 links, 4 joints
Links:
- removed link Link1
- removed link Link2
- removed link Link3
- removed link Link4
- removed link base_link
- added link gripper_Link1, mass 0.0024857; collision mesh filename=package://eg2_4b_description/meshes/gripper_Link1.STL; visual mesh filename=package://eg2_4b_description/meshes/gripper_Link1.STL
- added link gripper_Link2, mass 0.0044927; collision mesh filename=package://eg2_4b_description/meshes/gripper_Link2.STL; visual mesh filename=package://eg2_4b_description/meshes/gripper_Link2.STL
- added link gripper_Link3, mass 0.0024857; collision mesh filename=package://eg2_4b_description/meshes/gripper_Link3.STL; visual mesh filename=package://eg2_4b_description/meshes/gripper_Link3.STL
- added link gripper_Link4, mass 0.0044926; collision mesh filename=package://eg2_4b_description/meshes/gripper_Link4.STL; visual mesh filename=package://eg2_4b_description/meshes/gripper_Link4.STL
- added link gripper_base_link, mass 0.075349; collision mesh filename=package://eg2_4b_description/meshes/gripper_base_link.STL; visual mesh filename=package://eg2_4b_description/meshes/gripper_base_link.STL
Joints:
- removed joint joint1
- removed joint joint2
- removed joint joint3
- removed joint joint4
- added joint gripper_joint1: type revolute, parent gripper_base_link, child gripper_Link1, origin xyz=0 -0.04 0.09 rpy=0 0 0, axis 1 0 0, limit lower=0 upper=0.872 effort=0 velocity=0
- added joint gripper_joint2: type revolute, parent gripper_Link1, child gripper_Link2, origin xyz=0 0.022341 0.035565 rpy=0 0 0, axis -1 0 0, limit lower=0 upper=0.849 effort=0 velocity=0
- added joint gripper_joint3: type revolute, parent gripper_base_link, child gripper_Link3, origin xyz=0 0.04 0.09 rpy=0 0 0, axis -1 0 0, limit lower=0 upper=0.872 effort=0 velocity=0
- added joint gripper_joint4: type revolute, parent gripper_Link3, child gripper_Link4, origin xyz=0 -0.022341 0.035565 rpy=0 0 0, axis 1 0 0, limit lower=0 upper=0.849 effort=0 velocity=0

File: ros2_robot_ws/src/rm_moveit2_config/rm_65_config/config/rm_65_description.ros2_control.xacro (robot description, xacro)
@@ -50,4 +50,32 @@
                 <state_interface name="velocity"/>
             </joint>
+            <joint name="gripper_joint1">
+                <command_interface name="position"/>
+                <state_interface name="position">
+                  <param name="initial_value">0.0</param>
+                </state_interface>
+                <state_interface name="velocity"/>
+            </joint>
+            <joint name="gripper_joint2">
+                <command_interface name="position"/>
+                <state_interface name="position">
+                  <param name="initial_value">0.0</param>
+                </state_interface>
+                <state_interface name="velocity"/>
+            </joint>
+            <joint name="gripper_joint3">
+                <command_interface name="position"/>
+                <state_interface name="position">
+                  <param name="initial_value">0.0</param>
+                </state_interface>
+                <state_interface name="velocity"/>
+            </joint>
+            <joint name="gripper_joint4">
+                <command_interface name="position"/>
+                <state_interface name="position">
+                  <param name="initial_value">0.0</param>
+                </state_interface>
+                <state_interface name="velocity"/>
+            </joint>
         </ros2_control>
     </xacro:macro>

File: ros2_robot_ws/src/rm_moveit2_config/rm_65_config/config/rm_65_description.urdf.xacro (robot description, xacro)
@@ -3,5 +3,5 @@
     <xacro:arg name="initial_positions_file" default="initial_positions.yaml" />
     <!-- Import rm_65_description urdf file -->
-    <xacro:include filename="$(find rm_description)/urdf/rm_65.urdf" />
+    <xacro:include filename="$(find rm_description)/urdf/rm_65_w_gripper.urdf.xacro" />
     <!-- Import control_xacro -->
     <xacro:include filename="rm_65_description.ros2_control.xacro" />

Commit message: Setup basic MTC package

File: ros2_robot_ws/src/eg2_4b_description/urdf/eg2_4b_description.urdf (robot description, URDF)
Before this commit: robot eg2_4b_description, 5 links, 4 joints
Links:
- link gripper_Link1: geometry collision mesh filename=file://$(find eg2_4b_description)/meshes/gripper_Link1.STL; visual mesh filename=file://$(find eg2_4b_description)/meshes/gripper_Link1.STL
- link gripper_Link2: geometry collision mesh filename=file://$(find eg2_4b_description)/meshes/gripper_Link2.STL; visual mesh filename=file://$(find eg2_4b_description)/meshes/gripper_Link2.STL
- link gripper_Link3: geometry collision mesh filename=file://$(find eg2_4b_description)/meshes/gripper_Link3.STL; visual mesh filename=file://$(find eg2_4b_description)/meshes/gripper_Link3.STL
- link gripper_Link4: geometry collision mesh filename=file://$(find eg2_4b_description)/meshes/gripper_Link4.STL; visual mesh filename=file://$(find eg2_4b_description)/meshes/gripper_Link4.STL
- link gripper_base_link: geometry collision mesh filename=file://$(find eg2_4b_description)/meshes/gripper_base_link.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; visual mesh filename=file://$(find eg2_4b_description)/meshes/gripper_base_link.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
Joints:
- joint gripper_joint1: limit lower=0 upper=0.872 effort=0 velocity=0 -> lower=0 upper=0.872 effort=1.0 velocity=1.0
- joint gripper_joint2: limit lower=0 upper=0.849 effort=0 velocity=0 -> lower=0 upper=0.849 effort=1.0 velocity=1.0
- joint gripper_joint3: limit lower=0 upper=0.872 effort=0 velocity=0 -> lower=0 upper=0.872 effort=1.0 velocity=1.0
- joint gripper_joint4: limit lower=0 upper=0.849 effort=0 velocity=0 -> lower=0 upper=0.849 effort=1.0 velocity=1.0
