Commit message: Added custom pose interfaces and added camera mount to urdf

File: ros2_robot_ws/src/rm_description/urdf/rm_65_w_gripper.urdf.xacro (robot description, xacro)
@@ -1,10 +1,16 @@
 <?xml version="1.0" encoding="utf-8"?>
 <robot name="rm_65_with_gripper" xmlns:xacro="http://www.ros.org/wiki/xacro">
-  <xacro:include filename="$(find rm_description)/urdf/rm_65.urdf.xacro"/>
-  <xacro:include filename="$(find eg2_4b_description)/urdf/eg2_4b_description.urdf"/>
+  <xacro:include filename="$(find rm_description)/urdf/rm_65.urdf.xacro" />
+  <xacro:include filename="$(find eg2_4b_description)/urdf/eg2_4b_description.urdf" />
   <joint name="gripper_attach" type="fixed">
-    <parent link="Link6"/>
-    <child link="gripper_base_link"/>
-    <origin xyz="0 0 0.004" rpy="0 0 0"/>
+    <parent link="Link6" />
+    <child link="gripper_base_link" />
+    <origin xyz="0 0 0.004" rpy="0 0 0" />
+  </joint>
+  <link name="camera_bottom_screw_frame" />
+  <joint name="camera_joint" type="fixed">
+    <parent link="Link6" />
+    <child link="camera_bottom_screw_frame" />
+    <origin xyz="0.014 -0.0125 0.0475" rpy="0 0 0" />
   </joint>
 </robot>

Commit message: Verified main working up till before state machine

File: ros2_robot_ws/src/rm_description/urdf/rm_65_w_gripper.urdf.xacro (robot description, xacro)
@@ -2,5 +2,6 @@
 <robot name="rm_65_with_gripper" xmlns:xacro="http://www.ros.org/wiki/xacro">
   <xacro:include filename="$(find rm_description)/urdf/rm_65.urdf.xacro" />
-  <xacro:include filename="$(find eg2_4b_description)/urdf/eg2_4b_description.urdf" />
+  <xacro:include filename="$(find rm_description)/urdf/eg2_4b_description_patch.urdf" />
+  <xacro:include filename="$(find realsense2_description)/urdf/_d435.urdf.xacro" />
   <joint name="gripper_attach" type="fixed">
     <parent link="Link6" />
@@ -8,9 +9,7 @@
     <origin xyz="0 0 0.004" rpy="0 0 0" />
   </joint>
-  <link name="camera_bottom_screw_frame" />
-  <joint name="camera_joint" type="fixed">
-    <parent link="Link6" />
-    <child link="camera_bottom_screw_frame" />
+  <!-- Link to camera tf_tree -->
+  <xacro:sensor_d435 parent="Link6" name="camera" use_nominal_extrinsics="false">
     <origin xyz="0.014 -0.0125 0.0475" rpy="0 0 0" />
-  </joint>
+  </xacro:sensor_d435>
 </robot>

File: ros2_robot_ws/src/rm_moveit2_config/rm_65_w_gripper_config/config/rm_65_with_gripper.ros2_control.xacro (robot description, xacro)
@@ -1,82 +1,85 @@
 <?xml version="1.0"?>
 <robot xmlns:xacro="http://www.ros.org/wiki/xacro">
-    <xacro:macro name="rm_65_with_gripper_ros2_control" params="name initial_positions_file">
-        <xacro:property name="initial_positions" value="${load_yaml(initial_positions_file)['initial_positions']}"/>
-        <ros2_control name="${name}" type="system">
-            <hardware>
-                <!-- By default, set up controllers for simulation. This won't work on real hardware -->
-                <plugin>mock_components/GenericSystem</plugin>
-            </hardware>
-            <joint name="joint1">
-                <command_interface name="position"/>
-                <state_interface name="position">
-                  <param name="initial_value">${initial_positions['joint1']}</param>
-                </state_interface>
-                <state_interface name="velocity"/>
-            </joint>
-            <joint name="joint2">
-                <command_interface name="position"/>
-                <state_interface name="position">
-                  <param name="initial_value">${initial_positions['joint2']}</param>
-                </state_interface>
-                <state_interface name="velocity"/>
-            </joint>
-            <joint name="joint3">
-                <command_interface name="position"/>
-                <state_interface name="position">
-                  <param name="initial_value">${initial_positions['joint3']}</param>
-                </state_interface>
-                <state_interface name="velocity"/>
-            </joint>
-            <joint name="joint4">
-                <command_interface name="position"/>
-                <state_interface name="position">
-                  <param name="initial_value">${initial_positions['joint4']}</param>
-                </state_interface>
-                <state_interface name="velocity"/>
-            </joint>
-            <joint name="joint5">
-                <command_interface name="position"/>
-                <state_interface name="position">
-                  <param name="initial_value">${initial_positions['joint5']}</param>
-                </state_interface>
-                <state_interface name="velocity"/>
-            </joint>
-            <joint name="joint6">
-                <command_interface name="position"/>
-                <state_interface name="position">
-                  <param name="initial_value">${initial_positions['joint6']}</param>
-                </state_interface>
-                <state_interface name="velocity"/>
-            </joint>
-            <joint name="gripper_joint1">
-                <command_interface name="position"/>
-                <state_interface name="position">
-                  <param name="initial_value">${initial_positions['gripper_joint1']}</param>
-                </state_interface>
-                <state_interface name="velocity"/>
-            </joint>
-            <joint name="gripper_joint2">
-                <command_interface name="position"/>
-                <state_interface name="position">
-                  <param name="initial_value">${initial_positions['gripper_joint2']}</param>
-                </state_interface>
-                <state_interface name="velocity"/>
-            </joint>
-            <joint name="gripper_joint3">
-                <command_interface name="position"/>
-                <state_interface name="position">
-                  <param name="initial_value">${initial_positions['gripper_joint3']}</param>
-                </state_interface>
-                <state_interface name="velocity"/>
-            </joint>
-            <joint name="gripper_joint4">
-                <command_interface name="position"/>
-                <state_interface name="position">
-                  <param name="initial_value">${initial_positions['gripper_joint4']}</param>
-                </state_interface>
-                <state_interface name="velocity"/>
-            </joint>
-        </ros2_control>
-    </xacro:macro>
+  <xacro:macro name="rm_65_with_gripper_ros2_control" params="name initial_positions_file">
+    <xacro:property name="initial_positions"
+      value="${load_yaml(initial_positions_file)['initial_positions']}" />
+    <ros2_control name="${name}" type="system">
+      <hardware>
+        <!-- By default, set up controllers for simulation. This won't work on real hardware -->
+        <plugin>mock_components/GenericSystem</plugin>
+      </hardware>
+      <joint name="joint1">
+        <command_interface name="position" />
+        <state_interface name="position">
+          <param name="initial_value">${initial_positions['joint1']}</param>
+        </state_interface>
+        <state_interface name="velocity" />
+      </joint>
+      <joint name="joint2">
+        <command_interface name="position" />
+        <state_interface name="position">
+          <param name="initial_value">${initial_positions['joint2']}</param>
+        </state_interface>
+        <state_interface name="velocity" />
+      </joint>
+      <joint name="joint3">
+        <command_interface name="position" />
+        <state_interface name="position">
+          <param name="initial_value">${initial_positions['joint3']}</param>
+        </state_interface>
+        <state_interface name="velocity" />
+      </joint>
+      <joint name="joint4">
+        <command_interface name="position" />
+        <state_interface name="position">
+          <param name="initial_value">${initial_positions['joint4']}</param>
+        </state_interface>
+        <state_interface name="velocity" />
+      </joint>
+      <joint name="joint5">
+        <command_interface name="position" />
+        <state_interface name="position">
+          <param name="initial_value">${initial_positions['joint5']}</param>
+        </state_interface>
+        <state_interface name="velocity" />
+      </joint>
+      <joint name="joint6">
+        <command_interface name="position" />
+        <state_interface name="position">
+          <param name="initial_value">${initial_positions['joint6']}</param>
+        </state_interface>
+        <state_interface name="velocity" />
+      </joint>
+      <!--
+      <joint name="gripper_joint1">
+          <command_interface name="position"/>
+          <state_interface name="position">
+            <param name="initial_value">${initial_positions['gripper_joint1']}</param>
+          </state_interface>
+          <state_interface name="velocity"/>
+      </joint>
+      <joint name="gripper_joint2">
+          <command_interface name="position"/>
+          <state_interface name="position">
+            <param name="initial_value">${initial_positions['gripper_joint2']}</param>
+          </state_interface>
+          <state_interface name="velocity"/>
+      </joint>
+      <joint name="gripper_joint3">
+          <command_interface name="position"/>
+          <state_interface name="position">
+            <param name="initial_value">${initial_positions['gripper_joint3']}</param>
+          </state_interface>
+          <state_interface name="velocity"/>
+      </joint>
+      <joint name="gripper_joint4">
+          <command_interface name="position"/>
+          <state_interface name="position">
+            <param name="initial_value">${initial_positions['gripper_joint4']}</param>
+          </state_interface>
+          <state_interface name="velocity"/>
+      </joint>
+      -->
+    </ros2_control>
+  </xacro:macro>
 </robot>

File: ros2_robot_ws/src/rm_moveit2_config/rm_65_w_gripper_config/config/rm_65_with_gripper.urdf.xacro (robot description, xacro)
@@ -6,4 +6,7 @@
     <!-- Import control_xacro -->
     <xacro:include filename="rm_65_with_gripper.ros2_control.xacro" />
-    <xacro:rm_65_with_gripper_ros2_control name="FakeSystem" initial_positions_file="$(arg initial_positions_file)"/>
+    <!--
+    <xacro:rm_65_with_gripper_ros2_control name="FakeSystem"
+        initial_positions_file="$(arg initial_positions_file)" />
+    -->
 </robot>

Commit message: SM working up till tf transform

File: ros2_robot_ws/src/rm_description/urdf/rm_65_w_gripper.urdf.xacro (robot description, xacro)
@@ -7,9 +7,9 @@
     <parent link="Link6" />
     <child link="gripper_base_link" />
-    <origin xyz="0 0 0.004" rpy="0 0 0" />
+    <origin xyz="0 0 0.004" rpy="0 0 1.5708" />
   </joint>
-  <!-- Link to camera tf_tree -->
+  <!-- Link to camera tf_tree, past offset <origin xyz="0.014 -0.0125 0.0475" rpy="0 0 0" />-->
   <xacro:sensor_d435 parent="Link6" name="camera" use_nominal_extrinsics="false">
-    <origin xyz="0.014 -0.0125 0.0475" rpy="0 0 0" />
+    <origin xyz="-0.0125 0.0475 0.014" rpy="0 -1.5708 -1.5708" />
   </xacro:sensor_d435>
 </robot>

Commit message: Validated movement pipeline

File: ros2_robot_ws/src/rm_description/urdf/rm_65_w_gripper.urdf.xacro (robot description, xacro)
@@ -9,4 +9,10 @@
     <origin xyz="0 0 0.004" rpy="0 0 1.5708" />
   </joint>
+  <link name="grasp_frame" />
+  <joint name="grasp_frame_joint" type="fixed">
+    <parent link="Link6" />
+    <child link="grasp_frame" />
+    <origin xyz="0 0 0" rpy="0 0 3.1416" />
+  </joint>
   <!-- Link to camera tf_tree, past offset <origin xyz="0.014 -0.0125 0.0475" rpy="0 0 0" />-->
   <xacro:sensor_d435 parent="Link6" name="camera" use_nominal_extrinsics="false">

Commit message: Preemptive logic fixes for SM

File: ros2_robot_ws/src/rm_description/urdf/rm_65_w_gripper.urdf.xacro (robot description, xacro)
@@ -13,5 +13,5 @@
     <parent link="Link6" />
     <child link="grasp_frame" />
-    <origin xyz="0 0 0" rpy="0 0 3.1416" />
+    <origin xyz="0 0 0.1475" rpy="0 0 3.1416" />
   </joint>
   <!-- Link to camera tf_tree, past offset <origin xyz="0.014 -0.0125 0.0475" rpy="0 0 0" />-->

Commit message: Approach till final grasp

File: ros2_robot_ws/src/rm_description/urdf/rm_65_w_gripper.urdf.xacro (robot description, xacro)
@@ -13,5 +13,5 @@
     <parent link="Link6" />
     <child link="grasp_frame" />
-    <origin xyz="0 0 0.1475" rpy="0 0 3.1416" />
+    <origin xyz="0 0 0.1475" rpy="3.1416 0 1.5708 " />
   </joint>
   <!-- Link to camera tf_tree, past offset <origin xyz="0.014 -0.0125 0.0475" rpy="0 0 0" />-->
